Commit message: temp

File: urdf/gp100_comp.urdf (robot description, URDF)
Before this commit: robot archer_y6_gp100, 9 links, 8 joints
Links:
- link gp100_base_link: mass 0.21156702451304 -> 0.49249680
- link gp100_link_1: mass 0.0554322117046305 -> 0.02628607
- link gp100_link_2: mass 0.0554322115508225 -> 0.02628607
Joints:
- joint gp100_joint_1: axis -1 0 0 -> (none); limit lower=0 upper=0.7 effort=0 velocity=0 -> (none); origin xyz=0 -0.015 0.076799 rpy=0 0 0 -> xyz=0 -0.014 0.076799 rpy=0 0 0; type revolute -> fixed
- joint gp100_joint_2: axis 1 0 0 -> (none); limit lower=0 upper=0.7 effort=0 velocity=0 -> (none); origin xyz=0 0.015 0.076799 rpy=0 0 0 -> xyz=0 0.014 0.076799 rpy=0 0 0; type revolute -> fixed

Commit message: temp

File: urdf/gp100_comp.urdf (robot description, URDF)
Before this commit: robot archer_y6_gp100, 9 links, 8 joints
Links:
- link gp100_link_1: mass 0.02628607 -> 0.02438432
- link gp100_link_2: mass 0.02628607 -> 0.02438432

File: urdf/gp100_full.urdf (robot description, URDF)
Before this commit: robot archer_y6_gp100, 9 links, 8 joints
Links:
- link gp100_link_1: mass 0.02628607 -> 0.02438432
- link gp100_link_2: mass 0.02628607 -> 0.02438432
