Commit message: refactor(gr100*) gp100 -> gr100

File: urdf/gr100_comp.urdf (robot description, URDF)
Before this commit: robot archer_y6_gp100, 9 links, 8 joints
Links:
- removed link gp100_base_link
- removed link gp100_link_1
- removed link gp100_link_2
- added link grip_base_link, mass 0.49249680; collision mesh filename=package://hex_ros_urdf_archer_y6/meshes/gr100_base_link.STL; visual mesh filename=package://hex_ros_urdf_archer_y6/meshes/gr100_base_link.STL
- added link grip_link_1, mass 0.02438432; collision mesh filename=package://hex_ros_urdf_archer_y6/meshes/gr100_link_1.STL; visual mesh filename=package://hex_ros_urdf_archer_y6/meshes/gr100_link_1.STL
- added link grip_link_2, mass 0.02438432; collision mesh filename=package://hex_ros_urdf_archer_y6/meshes/gr100_link_2.STL; visual mesh filename=package://hex_ros_urdf_archer_y6/meshes/gr100_link_2.STL
Joints:
- removed joint gp100_joint_1
- removed joint gp100_joint_2
- added joint gr100_joint_1: type fixed, parent grip_base_link, child grip_link_1, origin xyz=0 -0.014 0.076799 rpy=0 0 0
- added joint gr100_joint_2: type fixed, parent grip_base_link, child grip_link_2, origin xyz=0 0.014 0.076799 rpy=0 0 0
- joint joint_6: child gp100_base_link -> grip_base_link

File: urdf/gr100_full.urdf (robot description, URDF)
Before this commit: robot archer_y6_gp100, 9 links, 8 joints
Links:
- removed link gp100_base_link
- removed link gp100_link_1
- removed link gp100_link_2
- added link grip_base_link, mass 0.49249680; collision mesh filename=package://hex_ros_urdf_archer_y6/meshes/gr100_base_link.STL; visual mesh filename=package://hex_ros_urdf_archer_y6/meshes/gr100_base_link.STL
- added link grip_link_1, mass 0.02438432; collision mesh filename=package://hex_ros_urdf_archer_y6/meshes/gr100_link_1.STL; visual mesh filename=package://hex_ros_urdf_archer_y6/meshes/gr100_link_1.STL
- added link grip_link_2, mass 0.02438432; collision mesh filename=package://hex_ros_urdf_archer_y6/meshes/gr100_link_2.STL; visual mesh filename=package://hex_ros_urdf_archer_y6/meshes/gr100_link_2.STL
Joints:
- removed joint gp100_joint_1
- removed joint gp100_joint_2
- added joint gr100_joint_1: type revolute, parent grip_base_link, child grip_link_1, origin xyz=0 -0.014 0.076799 rpy=0 0 0, axis -1 0 0, limit lower=0 upper=0.6 effort=0 velocity=0
- added joint gr100_joint_2: type revolute, parent grip_base_link, child grip_link_2, origin xyz=0 0.014 0.076799 rpy=0 0 0, axis 1 0 0, limit lower=0 upper=0.6 effort=0 velocity=0, mimic joint=gr100_joint_1 multiplier=1 offset=0
- joint joint_6: child gp100_base_link -> grip_base_link

Commit message: temp

File: urdf/gr100_comp.urdf (robot description, URDF)
Before this commit: robot archer_y6_gr100, 9 links, 8 joints
Links:
- removed link grip_base_link
- added link link_6, mass 0.49249680; collision mesh filename=package://hex_ros_urdf_archer_y6/meshes/gr100_base_link.STL; visual mesh filename=package://hex_ros_urdf_archer_y6/meshes/gr100_base_link.STL
Joints:
- removed joint gr100_joint_1
- removed joint gr100_joint_2
- added joint grip_joint_1: type fixed, parent link_6, child grip_link_1, origin xyz=0 -0.014 0.076799 rpy=0 0 0
- added joint grip_joint_2: type fixed, parent link_6, child grip_link_2, origin xyz=0 0.014 0.076799 rpy=0 0 0
- joint joint_6: child grip_base_link -> link_6

File: urdf/gr100_full.urdf (robot description, URDF)
Before this commit: robot archer_y6_gr100, 9 links, 8 joints
Links:
- removed link grip_base_link
- added link link_6, mass 0.49249680; collision mesh filename=package://hex_ros_urdf_archer_y6/meshes/gr100_base_link.STL; visual mesh filename=package://hex_ros_urdf_archer_y6/meshes/gr100_base_link.STL
Joints:
- removed joint gr100_joint_1
- removed joint gr100_joint_2
- added joint grip_joint_1: type revolute, parent link_6, child grip_link_1, origin xyz=0 -0.014 0.076799 rpy=0 0 0, axis -1 0 0, limit lower=0 upper=0.6 effort=0 velocity=0
- added joint grip_joint_2: type revolute, parent link_6, child grip_link_2, origin xyz=0 0.014 0.076799 rpy=0 0 0, axis 1 0 0, limit lower=0 upper=0.6 effort=0 velocity=0, mimic joint=grip_joint_1 multiplier=1 offset=0
- joint joint_6: child grip_base_link -> link_6
